File: fclub/fclub.kicad_sch (KiCad schematic)
At the start: 13 parts, among them SW1 SW_Push, U1 ATmega32U4-A, Y2 Crystal_GND24_Small

Commit message: a
Parts:
- added SW10, SW2, SW3, SW4, SW5, SW6, SW7, SW8, SW9: SW_Push_45deg, PCM_marbastlib-mx:SW_MX_1u, symbol Switch:SW_Push_45deg
- added U2: STM32F042K4Tx, Package_QFP:LQFP-32_7x7mm_P0.8mm, symbol MCU_ST_STM32F0:STM32F042K4Tx
Other:
- moved on the sheet: C1, C2, C3, C4, C5, C6, C7, R1, R2, R3, SW1, U1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

Commit message: passage stm
Parts:
- removed C6, C7: 22pF, symbol Device:C_Small
- removed R2, R3: 22, symbol Device:R_Small
- removed SW1: SW_Push, symbol Switch:SW_Push
- removed U1: ATmega32U4-A, Package_QFP:TQFP-44_10x10mm_P0.8mm, symbol MCU_Microchip_ATmega:ATmega32U4-A
- removed Y2: Crystal_GND24_Small, symbol Device:Crystal_GND24_Small
- added SW11: SW_Push, symbol Switch:SW_Push
- C1: value 1uF -> C_Small
- C2: value 0.1uF -> 1uF
- C3, C4: value 0.1uF -> 100nF
- C5: value 10uF -> 100nF
- R1: value 10k -> R_Small
Connections:
- net +5V: now also R1.1, U2.1 (VDD), U2.17 (VDDIO2), U2.5 (VDDA)
- net GND: now also U2.16 (VSS), U2.32 (VSSA), SW11.2; no longer R1.2
- net at C1.1: now also R1.2, U2.4 (NRST), SW11.1
Other:
- moved on the sheet: U2

Commit message: schematic fini
Parts:
- removed SW10: SW_Push_45deg, PCM_marbastlib-mx:SW_MX_1u, symbol Switch:SW_Push_45deg
- added D1, D2, D3, D4, D5, D6, D7, D8, D9: D, Diode_SMD:D_SOD-323_HandSoldering, symbol Device:D
- added J1: USB_C_Receptacle_USB2.0_14P, Connector_USB:USB_C_Receptacle_GCT_USB4105-xx-A_16P_TopMnt_Horizontal, symbol Connector:USB_C_Receptacle_USB2.0_14P
- added R2, R3: 5.1K, symbol Device:R_Small
- added SW1: SW_Push_45deg, PCM_marbastlib-mx:SW_MX_1u, symbol Switch:SW_Push_45deg
- C1: value C_Small -> 100nF
- R1: value R_Small -> 100K
Connections:
- net +5V: now also J1.A4 (VBUS), J1.A9 (VBUS), J1.B4 (VBUS), J1.B9 (VBUS)
- net GND: now also J1.A1 (GND), J1.A12 (GND), J1.B1 (GND), J1.B12 (GND), J1.S1 (SHIELD), R2.2, R3.2
- net at SW9.1: now also D9.2 (A)
- net col3: now reaches SW9.2
- net col3: now also SW3.2, SW6.2, U2.9 (PA3)
- net at SW5.1: now also D5.2 (A)
- net col2: now reaches SW5.2
- net col2: now also SW2.2, SW8.2, U2.8 (PA2)
- net at SW8.1: now also D8.2 (A)
- net at SW4.1: now also D4.2 (A)
- net col1: now reaches SW4.2
- net col1: now also SW7.2, U2.7 (PA1), SW1.2
- net at SW7.1: now also D7.2 (A)
- net at SW6.1: now also D6.2 (A)
- net row1: now reaches U2.10 (PA4)
- net row1: now also D1.1 (K), D2.1 (K), D3.1 (K)
- net row2: now reaches U2.11 (PA5)
- net row2: now also D4.1 (K), D5.1 (K), D6.1 (K)
- net row3: now reaches U2.12 (PA6)
- net row3: now also D7.1 (K), D8.1 (K), D9.1 (K)
- net D-: now reaches U2.21 (PA11)
- net D-: now also J1.A7 (D-), J1.B7 (D-)
- net D+: now reaches U2.22 (PA12)
- net D+: now also J1.A6 (D+), J1.B6 (D+)
- net at SW3.1: now also D3.2 (A)
- net at SW2.1: now also D2.2 (A)
- new net: J1.A5 (CC1), R2.1
- new net: D1.2 (A), SW1.1
- new net: J1.B5 (CC2), R3.1
Other:
- moved on the sheet: C1, C2, C3, C4, C5, R1, SW11, U2

Commit message: pcb fini
Parts:
- C1, C2, C3, C4, C5: footprint (none) -> Capacitor_SMD:C_0201_0603Metric_Pad0.64x0.40mm_HandSolder
- R1, R2, R3: footprint (none) -> Resistor_SMD:R_0201_0603Metric_Pad0.64x0.40mm_HandSolder
- SW11: footprint (none) -> random-keyboard-parts:SKQG-1155865
Changed lines of the file:
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@@
 			)
 		)
-		(property "Footprint" ""
+		(property "Footprint" "random-keyboard-parts:SKQG-1155865"
 			(at 198.12 59.69 0)
 			(effects
@@
 			)
 		)
-		(property "Footprint" ""
+		(property "Footprint" "Capacitor_SMD:C_0201_0603Metric_Pad0.64x0.40mm_HandSolder"
 			(at 182.88 59.69 0)
 			(effects
@@
 			)
 		)
-		(property "Footprint" ""
+		(property "Footprint" "Capacitor_SMD:C_0201_0603Metric_Pad0.64x0.40mm_HandSolder"
 			(at 184.15 92.71 0)
 			(effects
@@
 			)
 		)
-		(property "Footprint" ""
+		(property "Footprint" "Resistor_SMD:R_0201_0603Metric_Pad0.64x0.40mm_HandSolder"
 			(at 124.46 127 0)
 			(effects
@@
 			)
 		)
-		(property "Footprint" ""
+		(property "Footprint" "Capacitor_SMD:C_0201_0603Metric_Pad0.64x0.40mm_HandSolder"
 			(at 193.04 92.71 0)
 			(effects
@@
 			)
 		)
-		(property "Footprint" ""
+		(property "Footprint" "Capacitor_SMD:C_0201_0603Metric_Pad0.64x0.40mm_HandSolder"
 			(at 204.47 92.71 0)
 			(effects
@@
 			)
 		)
-		(property "Footprint" ""
+		(property "Footprint" "Capacitor_SMD:C_0201_0603Metric_Pad0.64x0.40mm_HandSolder"
 			(at 172.72 92.71 0)
 			(effects
@@
 			)
 		)
-		(property "Footprint" ""
+		(property "Footprint" "Resistor_SMD:R_0201_0603Metric_Pad0.64x0.40mm_HandSolder"
 			(at 187.96 45.72 0)
 			(effects
@@
 			)
 		)
-		(property "Footprint" ""
+		(property "Footprint" "Resistor_SMD:R_0201_0603Metric_Pad0.64x0.40mm_HandSolder"
 			(at 114.3 129.54 0)
 			(effects
